File: kira_flight_computer_v2.kicad_sch (KiCad schematic)
At the start: 3 parts, among them J7 Conn_01x04_Socket

Commit message: updates
Parts:
- added H1, H2, H3, H4: MountingHole_Pad, MountingHole:MountingHole_2.2mm_M2_Pad_TopBottom, symbol Mechanical:MountingHole_Pad
- TP1, TP2: footprint TestPoint:TestPoint_Pad_D2.0mm -> TestPoint:TestPoint_Pad_D1.0mm
Connections:
- net GND: now also H1.1, H2.1, H3.1, H4.1
