File: MCU.kicad_sch (KiCad schematic)
At the start: 22 parts, among them SW1 SW_SPST, U1 STM32F411VETx, Y1 Resonator

Commit message: updates
Parts:
- C1, C2, C8: footprint Capacitor_SMD:C_0603_1608Metric_Pad1.08x0.95mm_HandSolder -> Capacitor_SMD:C_0603_1608Metric
- Y1: footprint Crystal:Crystal_SMD_WE_IQXC-240-4Pin_1.2x1.0mm -> Crystal:Crystal_SMD_SeikoEpson_TSX3225-4Pin_3.2x2.5mm
Connections:
- net GPIO/PD7: now reaches U1.88 (PD7)
- net GPIO/PA15: no longer names the net of U1.77 (PA15)
Changed lines of the file:
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@@
 		)
 	)
-	(global_label "GPIO{slash}PA15"
+	(global_label "GPIO{slash}PD7"
 		(shape input)
-		(at 132.08 85.09 0)
-		(fields_autoplaced yes)
-		(effects
-			(font
-				(size 1.27 1.27)
-			)
-			(justify left)
+		(at 86.36 130.81 180)
+		(fields_autoplaced yes)
+		(effects
+			(font
+				(size 1.27 1.27)
+			)
+			(justify right)
 		)
 		(property "Intersheetrefs" "${INTERSHEET_REFS}"
-			(at 145.6486 85.09 0)
-			(effects
-				(font
-					(size 1.27 1.27)
-				)
-				(justify left)
+			(at 73.8195 130.81 0)
+			(effects
+				(font
+					(size 1.27 1.27)
+				)
+				(justify right)
 				(hide yes)
 			)
@@
 			)
 		)
-		(property "Footprint" "Crystal:Crystal_SMD_WE_IQXC-240-4Pin_1.2x1.0mm"
+		(property "Footprint" "Crystal:Crystal_SMD_SeikoEpson_TSX3225-4Pin_3.2x2.5mm"
 			(at 56.515 86.36 0)
 			(effects
@@
 			)
 		)
-		(property "Footprint" "Capacitor_SMD:C_0603_1608Metric_Pad1.08x0.95mm_HandSolder"
+		(property "Footprint" "Capacitor_SMD:C_0603_1608Metric"
 			(at 185.1152 34.29 0)
 			(effects
@@
 			)
 		)
-		(property "Footprint" "Capacitor_SMD:C_0603_1608Metric_Pad1.08x0.95mm_HandSolder"
+		(property "Footprint" "Capacitor_SMD:C_0603_1608Metric"
 			(at 197.8152 34.29 0)
 			(effects
@@
 			)
 		)
-		(property "Footprint" "Capacitor_SMD:C_0603_1608Metric_Pad1.08x0.95mm_HandSolder"
+		(property "Footprint" "Capacitor_SMD:C_0603_1608Metric"
 			(at 275.2852 34.29 0)
 			(effects

Commit message: Updatte
Parts:
- added C30: 100nF, Capacitor_SMD:C_0603_1608Metric, symbol Device:C
- added U8: USBLC6-2SC6, Package_TO_SOT_SMD:SOT-23-6, symbol Power_Protection:USBLC6-2SC6
Connections:
- net GND: now also C30.2, U8.2 (GND)
- net SERVO1: now also U8.4 (I/O2); no longer U1.90 (PB4)
- net SERVO2: now also U8.6 (I/O1); no longer U1.91 (PB5)
- new net: U1.91 (PB5), U8.1 (I/O1)
- new net: U1.90 (PB4), U8.3 (I/O2)
- new net +5V: C30.1, U8.5 (VBUS)
