File: Port_GPIO.kicad_sch (KiCad schematic)
At the start: 16 parts, among them J1 Conn_01x03_Pin, J10 Conn_01x06_Pin, J11 Conn_01x05_Pin, J2 Conn_01x03_Pin, J3 USB_C_Receptacle_USB2.0_14P, J4 Conn_01x06_Pin, J5 TC2030, J8 Conn_01x05_Pin, J9 Conn_01x06_Pin, U2 USBLC6-2SC6

Commit message: updates
Parts:
- C17, C18: value 10nF -> 100nF
- J11, J8: footprint Connector_JST:JST_GH_SM05B-GHS-TB_1x05-1MP_P1.25mm_Horizontal -> Connector_JST:JST_GH_BM05B-GHS-TBT_1x05-1MP_P1.25mm_Vertical
Connections:
- net GPIO/PA15 is gone; now on net GND: J11.1 (Pin_1)
- net +3.3V: now also J8.2 (Pin_2); no longer J8.4 (Pin_4)
- net +5V: now also J11.2 (Pin_2); no longer J11.4 (Pin_4)
- net GND: now also J8.1 (Pin_1); no longer J11.5 (Pin_5), J8.5 (Pin_5)
- net GPIO/PC8: now also J8.5 (Pin_5); no longer J8.1 (Pin_1)
- net UART1_RX: now also J8.4 (Pin_4); no longer J8.2 (Pin_2)
- net UART2_TX: now also J11.4 (Pin_4); no longer J11.2 (Pin_2)
- new net GPIO/PD7: J11.5 (Pin_5)
Other:
- moved on the sheet: C17, C18, J11, J8
Changed lines of the file:
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@@
 	)
 	(junction
-		(at 248.92 40.64)
+		(at 63.5 62.23)
 		(diameter 0)
 		(color 0 0 0 0)
 	)
 	(junction
-		(at 196.85 40.64)
+		(at 194.31 40.64)
 		(diameter 0)
 		(color 0 0 0 0)
 	)
 	(junction
-		(at 63.5 62.23)
+		(at 63.5 59.69)
 		(diameter 0)
 		(color 0 0 0 0)
 	)
 	(junction
-		(at 63.5 59.69)
+		(at 81.28 60.96)
 		(diameter 0)
 		(color 0 0 0 0)
 	)
 	(junction
-		(at 81.28 60.96)
+		(at 45.72 88.9)
 		(diameter 0)
 		(color 0 0 0 0)
 	)
 	(junction
-		(at 45.72 88.9)
+		(at 246.38 40.64)
 		(diameter 0)
 		(color 0 0 0 0)
@@
 	(wire
 		(pts
-			(xy 196.85 49.53) (xy 196.85 48.26)
+			(xy 194.31 49.53) (xy 194.31 48.26)
 		)
 		(stroke
@@
 	(wire
 		(pts
-			(xy 248.92 40.64) (xy 259.08 40.64)
-		)
-		(stroke
-			(width 0)
-			(type default)
-		)
-	)
-	(wire
-		(pts
 			(xy 205.74 43.18) (xy 205.74 49.53)
 		)
@@
 	(wire
 		(pts
-			(xy 248.92 29.21) (xy 248.92 40.64)
+			(xy 246.38 29.21) (xy 246.38 40.64)
 		)
 		(stroke
@@
 	(wire
 		(pts
-			(xy 196.85 40.64) (xy 207.01 40.64)
-		)
-		(stroke
-			(width 0)
-			(type default)
-		)
-	)
-	(wire
-		(pts
 			(xy 71.12 121.92) (xy 71.12 125.73)
 		)
@@
 	(wire
 		(pts
+			(xy 246.38 40.64) (xy 259.08 40.64)
+		)
+		(stroke
+			(width 0)
+			(type default)
+		)
+	)
+	(wire
+		(pts
 			(xy 71.12 143.51) (xy 71.12 138.43)
 		)
@@
 	(wire
 		(pts
-			(xy 196.85 29.21) (xy 196.85 40.64)
+			(xy 194.31 29.21) (xy 194.31 40.64)
 		)
 		(stroke
@@
 	(wire
 		(pts
-			(xy 248.92 49.53) (xy 248.92 48.26)
+			(xy 246.38 49.53) (xy 246.38 48.26)
 		)
 		(stroke
@@
 	(wire
 		(pts
+			(xy 194.31 40.64) (xy 207.01 40.64)
+		)
+		(stroke
+			(width 0)
+			(type default)
+		)
+	)
+	(wire
+		(pts
 			(xy 35.56 121.92) (xy 35.56 125.73)
 		)
@@
 		)
 	)
-	(global_label "GPIO{slash}PA15"
+	(global_label "GPIO{slash}PD7"
 		(shape input)
 		(at 240.03 106.68 180)
@@
 		)
 		(property "Intersheetrefs" "${INTERSHEET_REFS}"
-			(at 226.4614 106.68 0)
+			(at 227.4895 106.68 0)
 			(effects
 				(font
@@
 	(symbol
 		(lib_id "Connector:Conn_01x05_Pin")
-		(at 264.16 78.74 0)
-		(mirror y)
+		(at 264.16 78.74 180)
 		(unit 1)
 		(exclude_from_sim no)
@@
 		(on_board yes)
 		(dnp no)
-		(fields_autoplaced yes)
 		(property "Reference" "J8"
-			(at 265.43 77.4699 0)
+			(at 265.43 80.0101 0)
 			(effects
 				(font
@@
 		)
 		(property "Value" "Conn_01x05_Pin"
-			(at 265.43 80.0099 0)
+			(at 265.43 77.4701 0)
 			(effects
 				(font
@@
 			)
 		)
-		(property "Footprint" "Connector_JST:JST_GH_SM05B-GHS-TB_1x05-1MP_P1.25mm_Horizontal"
+		(property "Footprint" "Connector_JST:JST_GH_BM05B-GHS-TBT_1x05-1MP_P1.25mm_Vertical"
 			(at 264.16 78.74 0)
 			(effects
@@
 	(symbol
 		(lib_id "Device:C")
-		(at 248.92 44.45 0)
+		(at 246.38 44.45 0)
 		(unit 1)
 		(exclude_from_sim no)
@@
 		(fields_autoplaced yes)
 		(property "Reference" "C18"
-			(at 252.73 43.1799 0)
+			(at 250.19 43.1799 0)
 			(effects
 				(font
@@
 			)
 		)
-		(property "Value" "10nF"
-			(at 252.73 45.7199 0)
+		(property "Value" "100nF"
+			(at 250.19 45.7199 0)
 			(effects
 				(font
@@
 		)
 		(property "Footprint" "Capacitor_SMD:C_0603_1608Metric_Pad1.08x0.95mm_HandSolder"
-			(at 249.8852 48.26 0)
+			(at 247.3452 48.26 0)
 			(effects
 				(font
@@
 		)
 		(property "Datasheet" "~"
-			(at 248.92 44.45 0)
+			(at 246.38 44.45 0)
 			(effects
 				(font
@@
 		)
 		(property "Description" "Unpolarized capacitor"
-			(at 248.92 44.45 0)
+			(at 246.38 44.45 0)
 			(effects
 				(font
@@
 	(symbol
 		(lib_id "power:+3.3V")
-		(at 248.92 29.21 0)
+		(at 246.38 29.21 0)
 		(mirror y)
 		(unit 1)
@@
 		(dnp no)
 		(property "Reference" "#PWR020"
-			(at 248.92 33.02 0)
+			(at 246.38 33.02 0)
 			(effects
 				(font
@@
 		)
 		(property "Value" "+5V"
-			(at 248.92 24.13 0)
+			(at 246.38 24.13 0)
 			(effects
 				(font
@@
 		)
 		(property "Footprint" ""
-			(at 248.92 29.21 0)
+			(at 246.38 29.21 0)
 			(effects
 				(font
@@
 		)
 		(property "Datasheet" ""
-			(at 248.92 29.21 0)
+			(at 246.38 29.21 0)
 			(effects
 				(font
@@
 		)
 		(property "Description" "Power symbol creates a global label with name \"+3.3V\""
-			(at 248.92 29.21 0)
+			(at 246.38 29.21 0)
 			(effects
 				(font
@@
 	(symbol
 		(lib_id "power:+3.3V")
-		(at 196.85 29.21 0)
+		(at 194.31 29.21 0)
 		(mirror y)
 		(unit 1)
@@
 		(dnp no)
 		(property "Reference" "#PWR019"
-			(at 196.85 33.02 0)
+			(at 194.31 33.02 0)
 			(effects
 				(font
@@
 		)
 		(property "Value" "+5V"
-			(at 196.85 24.13 0)
+			(at 194.31 24.13 0)
 			(effects
 				(font
@@
 		)
 		(property "Footprint" ""
-			(at 196.85 29.21 0)
+			(at 194.31 29.21 0)
 			(effects
 				(font
@@
 		)
 		(property "Datasheet" ""
-			(at 196.85 29.21 0)
+			(at 194.31 29.21 0)
 			(effects
 				(font
@@
 		)
 		(property "Description" "Power symbol creates a global label with name \"+3.3V\""
-			(at 196.85 29.21 0)
+			(at 194.31 29.21 0)
 			(effects
 				(font
@@
 	(symbol
 		(lib_id "power:GND")
-		(at 248.92 49.53 0)
+		(at 246.38 49.53 0)
 		(unit 1)
 		(exclude_from_sim no)
@@
 		(fields_autoplaced yes)
 		(property "Reference" "#PWR025"
-			(at 248.92 55.88 0)
+			(at 246.38 55.88 0)
 			(effects
 				(font
@@
 		)
 		(property "Value" "GND"
-			(at 248.92 54.61 0)
+			(at 246.38 54.61 0)
 			(effects
 				(font
@@
 		)
 		(property "Footprint" ""
-			(at 248.92 49.53 0)
+			(at 246.38 49.53 0)
 			(effects
 				(font
@@
 		)
 		(property "Datasheet" ""
-			(at 248.92 49.53 0)
+			(at 246.38 49.53 0)
 			(effects
 				(font
@@
 		)
 		(property "Description" "Power symbol creates a global label with name \"GND\" , ground"
-			(at 248.92 49.53 0)
+			(at 246.38 49.53 0)
 			(effects
 				(font
@@
 	(symbol
 		(lib_id "Connector:Conn_01x05_Pin")
-		(at 259.08 111.76 0)
-		(mirror y)
+		(at 259.08 111.76 180)
 		(unit 1)
 		(exclude_from_sim no)
@@
 		(on_board yes)
 		(dnp no)
-		(fields_autoplaced yes)
 		(property "Reference" "J11"
-			(at 260.35 110.4899 0)
+			(at 260.35 113.0301 0)
 			(effects
 				(font
@@
 		)
 		(property "Value" "Conn_01x05_Pin"
-			(at 260.35 113.0299 0)
+			(at 260.35 110.4901 0)
 			(effects
 				(font
@@
 			)
 		)
-		(property "Footprint" "Connector_JST:JST_GH_SM05B-GHS-TB_1x05-1MP_P1.25mm_Horizontal"
+		(property "Footprint" "Connector_JST:JST_GH_BM05B-GHS-TBT_1x05-1MP_P1.25mm_Vertical"
 			(at 259.08 111.76 0)
 			(effects
@@
 	(symbol
 		(lib_id "Device:C")
-		(at 196.85 44.45 0)
+		(at 194.31 44.45 0)
 		(unit 1)
 		(exclude_from_sim no)
@@
 		(fields_autoplaced yes)
 		(property "Reference" "C17"
-			(at 200.66 43.1799 0)
+			(at 198.12 43.1799 0)
 			(effects
 				(font
@@
 			)
 		)
-		(property "Value" "10nF"
-			(at 200.66 45.7199 0)
+		(property "Value" "100nF"
+			(at 198.12 45.7199 0)
 			(effects
 				(font
@@
 		)
 		(property "Footprint" "Capacitor_SMD:C_0603_1608Metric_Pad1.08x0.95mm_HandSolder"
-			(at 197.8152 48.26 0)
+			(at 195.2752 48.26 0)
 			(effects
 				(font
@@
 		)
 		(property "Datasheet" "~"
-			(at 196.85 44.45 0)
+			(at 194.31 44.45 0)
 			(effects
 				(font
@@
 		)
 		(property "Description" "Unpolarized capacitor"
-			(at 196.85 44.45 0)
+			(at 194.31 44.45 0)
 			(effects
 				(font
@@
 	(symbol
 		(lib_id "power:GND")
-		(at 196.85 49.53 0)
+		(at 194.31 49.53 0)
 		(unit 1)
 		(exclude_from_sim no)
@@
 		(fields_autoplaced yes)
 		(property "Reference" "#PWR023"
-			(at 196.85 55.88 0)
+			(at 194.31 55.88 0)
 			(effects
 				(font
@@
 		)
 		(property "Value" "GND"
-			(at 196.85 54.61 0)
+			(at 194.31 54.61 0)
 			(effects
 				(font
@@
 		)
 		(property "Footprint" ""
-			(at 196.85 49.53 0)
+			(at 194.31 49.53 0)
 			(effects
 				(font
@@
 		)
 		(property "Datasheet" ""
-			(at 196.85 49.53 0)
+			(at 194.31 49.53 0)
 			(effects
 				(font
@@
 		)
 		(property "Description" "Power symbol creates a global label with name \"GND\" , ground"
-			(at 196.85 49.53 0)
+			(at 194.31 49.53 0)
 			(effects
 				(font

Commit message: Updatte
Parts:
- added C31: 100nF, Capacitor_SMD:C_0603_1608Metric_Pad1.08x0.95mm_HandSolder, symbol Device:C
Connections:
- net GND: now also C31.2
- net VBUS: now also C31.1
Other:
- moved on the sheet: R3
