File: kira_flight_computer_v2.kicad_pcb (KiCad board)
At the start: 4 copper layers, 53 x 103 mm, 74 parts, among them IC1 SC4216HSETRT, J1 Conn_01x03_Pin, J10 Conn_01x06_Pin, J11 Conn_01x05_Pin, J2 Conn_01x03_Pin, J3 USB_C_Receptacle_USB2.0_14P, J4 Conn_01x06_Pin, J5 TC2030, J7 Conn_01x04_Socket, J8 Conn_01x05_Pin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

Commit message: Add via stitching
Routing:
- net VDDIO: track 294.6 -> 317.3 mm, vias 44 -> 40
- net GND: track 145.2 -> 158.0 mm, vias 63 -> 229
- net +5V: track 141.5 -> 133.1 mm
- added copper zone on B.Cu, net +5V
Other:
- board text added: "+3V3"
- board text added: "CLK"
- board text added: "CS"
- board text added: "MISO"
- board text added: "MOSI"
- board text added: "SPI3"
- board text added: "SPI4"
- board text added: "SPI5"

Commit message: updates
Parts:
- added H1: MountingHole_Pad, MountingHole:MountingHole_2.2mm_M2_Pad_TopBottom, F.Cu at (65.2, 177.1)
- added H2: MountingHole_Pad, MountingHole:MountingHole_2.2mm_M2_Pad_TopBottom, F.Cu at (112.2, 177.1)
- added H3: MountingHole_Pad, MountingHole:MountingHole_2.2mm_M2_Pad_TopBottom, F.Cu at (112.2, 80.1)
- added H4: MountingHole_Pad, MountingHole:MountingHole_2.2mm_M2_Pad_TopBottom, F.Cu at (65.2, 80.1)
- C1, C2, C8: footprint Capacitor_SMD:C_0603_1608Metric_Pad1.08x0.95mm_HandSolder -> Capacitor_SMD:C_0603_1608Metric
- C17, C18: value 10nF -> 100nF
- J11, J8: footprint Connector_JST:JST_GH_SM05B-GHS-TB_1x05-1MP_P1.25mm_Horizontal -> Connector_JST:JST_GH_BM05B-GHS-TBT_1x05-1MP_P1.25mm_Vertical
- TP1, TP2, TP3, TP4: footprint TestPoint:TestPoint_Pad_D2.0mm -> TestPoint:TestPoint_Pad_D1.0mm
- Y1: footprint Crystal:Crystal_SMD_WE_IQXC-240-4Pin_1.2x1.0mm -> Crystal:Crystal_SMD_SeikoEpson_TSX3225-4Pin_3.2x2.5mm
- moved R11 11.7 mm to (73.1, 131.3)
- moved R10 10.5 mm to (73.1, 129.3)
- moved Y1 6.21 mm to (109.1, 139.0), turned to 0 degrees
- moved C1 3.60 mm to (103.1, 141.2)
- moved C16 3.60 mm to (80.8, 141.9)
- moved C25 3.60 mm to (107.5, 149.9)
- moved C26 3.60 mm to (104.2, 146.6)
- moved C28 3.60 mm to (91.6, 151.4)
- moved C29 3.60 mm to (88.8, 154.5)
- moved C3 3.60 mm to (103.1, 133.5)
- moved C9 3.60 mm to (103.1, 129.5)
- moved J1 3.60 mm to (84.1, 164.2)
- moved J11 3.60 mm to (69.5, 153.7), turned to 90 degrees
- moved J2 3.60 mm to (96.3, 164.2)
- moved J8 3.60 mm to (69.5, 142.0), turned to 90 degrees
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Connections:
- IC1 pad 9: unconnected-(IC1-EP-Pad9) -> GND
- J11 pad 1: unconnected-(J11-Pin_1-Pad1) -> GND
- J11 pad 2: /MCU/UART2_RX -> +5V
- J11 pad 4: +5V -> /MCU/UART2_RX
- J11 pad 5: GND -> GPIO/PD7
- J8 pad 1: GPIO/PC8 -> GND
- J8 pad 2: /MCU/UART1_TX -> VDDIO
- J8 pad 4: VDDIO -> /MCU/UART1_TX
- J8 pad 5: GND -> GPIO/PC8
- U1 pad 88: unconnected-(U1-PD7-Pad88) -> GPIO/PD7
Routing:
- net VDDIO: track 317.3 -> 211.1 mm, vias 40 -> 87
- net +5V: track 133.1 -> 69.8 mm, vias 1 -> 2
- net GPIO/PD7: track 0.00 -> 27.1 mm, vias 0 -> 2
- net Net-(U1-PH1): track 3.21 -> 11.3 mm
- net GND: track 158.0 -> 150.9 mm, vias 229 -> 260
- net Net-(U1-PH0): track 4.48 -> 9.53 mm
- net /MCU/UART2_RX: track 27.4 -> 26.3 mm
- net /Flash&Storage/I2C_SDA: track 14.4 -> 15.4 mm
- net /MCU/UART2_TX: track 26.6 -> 25.6 mm
- net /Flash&Storage/I2C_SCL: track 14.1 -> 14.7 mm
- added copper zone on B.Cu, net GND
- added copper zone on F.Cu, net GND
- added copper zone on In2.Cu, net VDDIO
Other:
- outline, holes or cut-outs redrawn

Commit message: Add Borderr
Parts:
- moved C17 9.17 mm to (92.9, 168.0)
- moved C18 9.17 mm to (105.1, 168.0)
- moved J1 8.13 mm to (89.2, 170.6)
- moved J2 8.13 mm to (101.3, 170.6)
- moved J3 7.07 mm to (77.0, 176.5)
- moved R5 7.07 mm to (79.7, 170.3)
- moved R3 7.07 mm to (74.3, 170.3)
- moved U2 7.07 mm to (76.9, 167.2)
- moved R4 3.44 mm to (70.5, 170.5)
- moved D1 3.44 mm to (70.5, 174.3)
Routing:
- net +5V: track 69.8 -> 155.9 mm
- net GND: track 150.9 -> 138.7 mm, vias 260 -> 317
- net /Ports_GPIO/SIG_CH2: track 21.1 -> 29.6 mm
- net /Ports_GPIO/D+: track 25.8 -> 33.3 mm
- net /Ports_GPIO/D-: track 26.7 -> 34.0 mm
- net VDDIO: track 211.1 -> 207.8 mm, vias 87 -> 88
- net /Ports_GPIO/SIG_CH1: track 24.7 -> 27.9 mm
- net VBUS: track 23.2 -> 20.4 mm, vias 0 -> 1
Other:
- outline, holes or cut-outs redrawn
- board text added: "SIG VCC GND"
- board text removed: "S V G"

Commit message: Updatte
Parts:
- added C30: 100nF, Capacitor_SMD:C_0603_1608Metric, F.Cu at (93.4, 163.6)
- added C31: 100nF, Capacitor_SMD:C_0603_1608Metric_Pad1.08x0.95mm_HandSolder, F.Cu at (79.7, 167.2)
- added U8: USBLC6-2SC6, Package_TO_SOT_SMD:SOT-23-6, F.Cu at (93.4, 160.3)
Connections:
- U1 pad 90: /Ports_GPIO/SIG_CH1 -> Net-(U1-PB4)
- U1 pad 91: /Ports_GPIO/SIG_CH2 -> Net-(U1-PB5)
Routing:
- net /Ports_GPIO/SIG_CH2: track 29.6 -> 12.0 mm
- net /Ports_GPIO/SIG_CH1: track 27.9 -> 10.5 mm
- net Net-(U1-PB5): track 0.00 -> 15.3 mm
- net Net-(U1-PB4): track 0.00 -> 15.1 mm
- net GND: track 138.7 -> 141.9 mm, vias 317 -> 309
- net +5V: track 155.9 -> 157.2 mm
- net VDDIO: track 207.8 -> 206.9 mm
- net VBUS: track 20.4 -> 21.1 mm, vias 1 -> 0
